Commit message: Added rtabmap
Signed-off-by: Gonzalo de Pedro <gonzalo@depedro.com.ar>

File: urdf/sjtu_drone.urdf (robot description, URDF)
Before this commit: robot sjtu_drone, 1 links, 0 joints
Links:
- added link camera_link
Joints:
- added joint base_to_right_leg: type fixed, parent base_link, child camera_link, origin rpy=-1.6 0 -1.6
